Commit message: Update robot.urdf

File: src/playground/urdf/robot.urdf (robot description, URDF)
Before this commit: robot mobile_robot, 6 links, 5 joints
Links:
- link base_link: geometry collision box size=0.5 0.3 0.2; visual box size=0.5 0.3 0.2
Joints:
- joint camera_joint: origin xyz=0.25 0 0.1 rpy=0 0 0 -> xyz=0.25 0 0.125 rpy=0 0 0
- joint caster_wheel_joint: origin xyz=-0.2 0 -0.05 rpy=0 0 0 -> xyz=-0.2 0 -0.1 rpy=0 0 0
- joint laser_joint: origin xyz=0 0 0.06 rpy=0 0 0 -> xyz=0 0 0.12 rpy=0 0 0
- joint left_wheel_joint: origin xyz=0.2 0.175 0 rpy=0 0 0 -> xyz=0.1 0.175 -0.05 rpy=0 0 0
- joint right_wheel_joint: origin xyz=0.2 -0.175 0 rpy=0 0 0 -> xyz=0.1 -0.175 -0.05 rpy=0 0 0
